File: DMH_Logic_PANEL/DMH_Logic_PANEL.kicad_pcb (KiCad board)
At the start: 2 copper layers, 50 x 200 mm, 5 parts, among them J0 Panel_GND_Solder_Wire_Pad

Commit message: Panel draft
Parts:
- removed J0: Panel_GND_Solder_Wire_Pad, SynthStuff:Panel_GND_SolderWirePad_5x10mm
- added H10: NOR K[Q'], SynthStuff:Jack_6.35mm_Cutout_Output_v6, F.Cu at (91.5, 153.2)
- added H11: FF 1, SynthStuff:Toggle_Switch_TE_Cutout, F.Cu at (58.5, 116.2)
- added H12: NOT A, SynthStuff:Jack_6.35mm_Cutout_v3, F.Cu at (75.0, 116.2)
- added H13: NOT A', SynthStuff:Jack_6.35mm_Cutout_Output_v6, F.Cu at (91.5, 116.2)
- added H14: FF 2, SynthStuff:Toggle_Switch_TE_Cutout, F.Cu at (58.5, 171.8)
- added H15: NOR E, SynthStuff:Jack_6.35mm_Cutout_v3, F.Cu at (58.5, 190.2)
- added H16: NOR G, SynthStuff:Jack_6.35mm_Cutout_v3, F.Cu at (58.5, 208.8)
- added H17: NOT B, SynthStuff:Jack_6.35mm_Cutout_v3, F.Cu at (75.0, 171.8)
- added H18: NOR F, SynthStuff:Jack_6.35mm_Cutout_v3, F.Cu at (75.0, 190.2)
- added H19: NOR H, SynthStuff:Jack_6.35mm_Cutout_v3, F.Cu at (75.0, 208.8)
- added H20: NOT B', SynthStuff:Jack_6.35mm_Cutout_Output_v6, F.Cu at (91.5, 171.8)
- added H21: NOR L[Q], SynthStuff:Jack_6.35mm_Cutout_Output_v6, F.Cu at (91.5, 190.2)
- added H22: NOR M[Q'], SynthStuff:Jack_6.35mm_Cutout_Output_v6, F.Cu at (91.5, 208.8)
- added H23: Switch, SynthStuff:Toggle_Switch_TE_Cutout, F.Cu at (58.5, 60.8)
- added H24: NAND A, SynthStuff:Jack_6.35mm_Cutout_v3, F.Cu at (58.5, 79.2)
- added H25: NAND C, SynthStuff:Jack_6.35mm_Cutout_v3, F.Cu at (58.5, 97.8)
- added H26: NOT C, SynthStuff:Jack_6.35mm_Cutout_v3, F.Cu at (75.0, 60.8)
- added H27: NAND B, SynthStuff:Jack_6.35mm_Cutout_v3, F.Cu at (75.0, 79.2)
- added H28: NAND D, SynthStuff:Jack_6.35mm_Cutout_v3, F.Cu at (75.0, 97.8)
- added H29: NOT C', SynthStuff:Jack_6.35mm_Cutout_Output_v6, F.Cu at (91.5, 60.8)
- added H30: NAND J, SynthStuff:Jack_6.35mm_Cutout_Output_v6, F.Cu at (91.5, 79.2)
- added H31: NAND K, SynthStuff:Jack_6.35mm_Cutout_Output_v6, F.Cu at (91.5, 97.8)
- added H5: NOR A, SynthStuff:Jack_6.35mm_Cutout_v3, F.Cu at (58.5, 134.8)
- added H6: NOR B, SynthStuff:Jack_6.35mm_Cutout_v3, F.Cu at (75.0, 134.8)
- added H7: NOR J[Q], SynthStuff:Jack_6.35mm_Cutout_Output_v6, F.Cu at (91.5, 134.8)
- added H8: NOR C, SynthStuff:Jack_6.35mm_Cutout_v3, F.Cu at (58.5, 153.2)
- added H9: NOR D, SynthStuff:Jack_6.35mm_Cutout_v3, F.Cu at (75.0, 153.2)
Other:
- board text added: "CMOS"
- board text added: "Logic"
- board text removed: "Module Name"
- board text removed: "TYPE"
