File: DMH_Logic_PANEL/DMH_Logic_PANEL.kicad_sch (KiCad schematic)
At the start: 5 parts, among them J0 Panel_GND_Solder_Wire_Pad

Commit message: Panel draft
Parts:
- added H10: NOR K[Q'], SynthStuff:Jack_6.35mm_Cutout_Output_v6, symbol SynthStuff:MountingHole_Jack6.35mm_Output_v2
- added H11: FF 1, SynthStuff:Toggle_Switch_TE_Cutout, symbol SynthStuff:MountingHole_ToggleSwitch
- added H12: NOT A, SynthStuff:Jack_6.35mm_Cutout_v3, symbol SynthStuff:MountingHole_Jack6.35mm_v2
- added H13: NOT A', SynthStuff:Jack_6.35mm_Cutout_Output_v6, symbol SynthStuff:MountingHole_Jack6.35mm_Output_v2
- added H14: FF 2, SynthStuff:Toggle_Switch_TE_Cutout, symbol SynthStuff:MountingHole_ToggleSwitch
- added H15: NOR E, SynthStuff:Jack_6.35mm_Cutout_v3, symbol SynthStuff:MountingHole_Jack6.35mm_v2
- added H16: NOR G, SynthStuff:Jack_6.35mm_Cutout_v3, symbol SynthStuff:MountingHole_Jack6.35mm_v2
- added H17: NOT B, SynthStuff:Jack_6.35mm_Cutout_v3, symbol SynthStuff:MountingHole_Jack6.35mm_v2
- added H18: NOR F, SynthStuff:Jack_6.35mm_Cutout_v3, symbol SynthStuff:MountingHole_Jack6.35mm_v2
- added H19: NOR H, SynthStuff:Jack_6.35mm_Cutout_v3, symbol SynthStuff:MountingHole_Jack6.35mm_v2
- added H20: NOT B', SynthStuff:Jack_6.35mm_Cutout_Output_v6, symbol SynthStuff:MountingHole_Jack6.35mm_Output_v2
- added H21: NOR L[Q], SynthStuff:Jack_6.35mm_Cutout_Output_v6, symbol SynthStuff:MountingHole_Jack6.35mm_Output_v2
- added H22: NOR M[Q'], SynthStuff:Jack_6.35mm_Cutout_Output_v6, symbol SynthStuff:MountingHole_Jack6.35mm_Output_v2
- added H23: Switch, SynthStuff:Toggle_Switch_TE_Cutout, symbol SynthStuff:MountingHole_ToggleSwitch
- added H24: NAND A, SynthStuff:Jack_6.35mm_Cutout_v3, symbol SynthStuff:MountingHole_Jack6.35mm_v2
- added H25: NAND C, SynthStuff:Jack_6.35mm_Cutout_v3, symbol SynthStuff:MountingHole_Jack6.35mm_v2
- added H26: NOT C, SynthStuff:Jack_6.35mm_Cutout_v3, symbol SynthStuff:MountingHole_Jack6.35mm_v2
- added H27: NAND B, SynthStuff:Jack_6.35mm_Cutout_v3, symbol SynthStuff:MountingHole_Jack6.35mm_v2
- added H28: NAND D, SynthStuff:Jack_6.35mm_Cutout_v3, symbol SynthStuff:MountingHole_Jack6.35mm_v2
- added H29: NOT C', SynthStuff:Jack_6.35mm_Cutout_Output_v6, symbol SynthStuff:MountingHole_Jack6.35mm_Output_v2
- added H30: NAND J, SynthStuff:Jack_6.35mm_Cutout_Output_v6, symbol SynthStuff:MountingHole_Jack6.35mm_Output_v2
- added H31: NAND K, SynthStuff:Jack_6.35mm_Cutout_Output_v6, symbol SynthStuff:MountingHole_Jack6.35mm_Output_v2
- added H5: NOR A, SynthStuff:Jack_6.35mm_Cutout_v3, symbol SynthStuff:MountingHole_Jack6.35mm_v2
- added H6: NOR B, SynthStuff:Jack_6.35mm_Cutout_v3, symbol SynthStuff:MountingHole_Jack6.35mm_v2
- added H7: NOR J[Q], SynthStuff:Jack_6.35mm_Cutout_Output_v6, symbol SynthStuff:MountingHole_Jack6.35mm_Output_v2
- added H8: NOR C, SynthStuff:Jack_6.35mm_Cutout_v3, symbol SynthStuff:MountingHole_Jack6.35mm_v2
- added H9: NOR D, SynthStuff:Jack_6.35mm_Cutout_v3, symbol SynthStuff:MountingHole_Jack6.35mm_v2
- J0: now not fitted
Connections:
- net GND: now also H10.1, H11.1, H12.1, H13.1, H14.1, H15.1, H16.1, H17.1, H18.1, H19.1, H20.1, H21.1, H22.1, H23.1, H24.1, H25.1, H26.1, H27.1, H28.1, H29.1, H30.1, H31.1, H5.1, H6.1, H7.1, H8.1, H9.1
Other:
- moved on the sheet: H1, H2, H3, H4
